File: PCB_PAMI_2025-2026/_autosave-PCB_PAMI_2025-2026.kicad_pcb (KiCad board)
At the start: 2 copper layers, 125 x 84 mm, 63 parts, among them J1 BAU, J10 MOTOR 4, J11 COMM_inter_mcu, J12 USB_C_Receptacle_USB2.0_16P, J13 BOOST_OUT, J2 BAT+, J3 VIN_Connector, J4 BAT-, J6 BOOST_IN, J7 MOTOR 3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

Commit message: correction emplacement batterie
Routing:
- net GND: track 108.5 -> 105.7 mm, vias 30 -> 29
Other:
- outline, holes or cut-outs redrawn
Changed lines of the file:
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@@
 	)
 	(gr_rect
-		(start 94 35.9)
-		(end 98 43.9)
+		(start 87.44 36.64)
+		(end 97.98 40.64)
 		(stroke
 			(width 0.2)
@@
 	)
 	(gr_rect
-		(start 94 68)
-		(end 98 76)
+		(start 87.44 69.66)
+		(end 97.98 73.66)
 		(stroke
 			(width 0.2)
@@
 	)
 	(segment
-		(start 137.16 60.96)
-		(end 137.16 58.24)
-		(width 1.5)
-		(layer "F.Cu")
-		(net 2)
-	)
-	(segment
 		(start 55.43 93.75)
 		(end 57.15 93.75)
@@
 		(net 2)
 	)
-	(segment
-		(start 137.16 58.24)
-		(end 137.2 58.2)
-		(width 1.5)
-		(layer "F.Cu")
-		(net 2)
-	)
 	(via
 		(at 73.5 67.7)
@@
 	)
 	(via
-		(at 137.2 58.2)
-		(size 0.6)
-		(drill 0.3)
-		(layers "F.Cu" "B.Cu")
-		(net 2)
-	)
-	(via
 		(at 115 44.1)
 		(size 0.6)
@@
 	(segment
 		(start 158.685 45.46)
-		(end 144.361 59.784)
+		(end 145.545 58.6)
 		(width 0.25)
 		(layer "B.Cu")
@@
 	)
 	(segment
-		(start 144.361 59.784)
-		(end 79.096 59.784)
+		(start 80.28 58.6)
+		(end 76.27 62.61)
 		(width 0.25)
 		(layer "B.Cu")
@@
 	)
 	(segment
-		(start 79.096 59.784)
-		(end 76.27 62.61)
+		(start 145.545 58.6)
+		(end 80.28 58.6)
 		(width 0.25)
 		(layer "B.Cu")
